File: board/board.kicad_pcb (KiCad board)
At the start: 2 copper layers, 21 x 13 mm, 1 part

Commit message: initial
Parts:
- added D1: LED, LED_SMD:LED_0603_1608Metric, F.Cu at (154.6, 95.0)
- added D2: LED, LED_SMD:LED_0603_1608Metric, F.Cu at (151.1, 95.0)
- added D3: LED, LED_SMD:LED_0603_1608Metric, F.Cu at (148.1, 95.0)
- added D4: LED, LED_SMD:LED_0603_1608Metric, F.Cu at (154.6, 98.0)
- added D5: LED, LED_SMD:LED_0603_1608Metric, F.Cu at (151.1, 98.1)
- added D6: LED, LED_SMD:LED_0603_1608Metric, F.Cu at (148.0, 98.0)
- added J1: 011_GPIO, on_edge:on_edge_2x05_host, F.Cu at (161.0, 96.5)
- added J2: 011_GPIO, on_edge:on_edge_2x05_device, F.Cu at (140.0, 96.5)
- added Q1: 2N7002K, Package_TO_SOT_SMD:SOT-23, F.Cu at (154.3, 91.8)
- added Q2: 2N7002K, Package_TO_SOT_SMD:SOT-23, F.Cu at (150.5, 91.8)
- added Q3: 2N7002K, Package_TO_SOT_SMD:SOT-23, F.Cu at (146.7, 91.8)
- added Q4: 2N7002K, Package_TO_SOT_SMD:SOT-23, F.Cu at (154.4, 101.2)
- added Q5: 2N7002K, Package_TO_SOT_SMD:SOT-23, F.Cu at (150.5, 101.2)
- added Q6: 2N7002K, Package_TO_SOT_SMD:SOT-23, F.Cu at (146.7, 101.2)
- added R1: 100R, Resistor_SMD:R_0603_1608Metric, F.Cu at (152.9, 95.0)
- added R2: 100R, Resistor_SMD:R_0603_1608Metric, F.Cu at (149.6, 95.0)
- added R3: 100R, Resistor_SMD:R_0603_1608Metric, F.Cu at (146.6, 95.0)
- added R4: 100R, Resistor_SMD:R_0603_1608Metric, F.Cu at (152.9, 98.0)
- added R5: 100R, Resistor_SMD:R_0603_1608Metric, F.Cu at (149.6, 98.0)
- added R6: 100R, Resistor_SMD:R_0603_1608Metric, F.Cu at (146.5, 98.0)
- LOGO1: moved to B.Cu
- moved LOGO1 0.70 mm to (150.7, 99.2), turned to 180 degrees
Routing:
- net GND: track 0.00 -> 40.7 mm
- net Net-(J1-GPIO4): track 0.00 -> 30.8 mm, vias 0 -> 1
- net Net-(J1-3.3V): track 0.00 -> 27.9 mm, vias 0 -> 1
- net Net-(J1-GPIO2): track 0.00 -> 27.6 mm, vias 0 -> 2
- net Net-(J1-GPIO5): track 0.00 -> 22.9 mm, vias 0 -> 1
- net Net-(J1-GPIO1): track 0.00 -> 21.7 mm, vias 0 -> 3
- net Net-(J1-GPIO3): track 0.00 -> 20.3 mm, vias 0 -> 3
- net Net-(J1-GPIO0): track 0.00 -> 18.8 mm, vias 0 -> 3
- net Net-(J1-5V): track 0.00 -> 16.2 mm
- net Net-(J1-GND-Pad8): track 0.00 -> 16.1 mm
- net Net-(D4-K): track 0.00 -> 7.80 mm
- net Net-(D2-K): track 0.00 -> 5.68 mm
- net Net-(D3-K): track 0.00 -> 5.38 mm
- net Net-(D6-K): track 0.00 -> 4.91 mm
- net Net-(D5-K): track 0.00 -> 4.41 mm
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Other:
- outline, holes or cut-outs redrawn
- board text added: "osf.100"
- board text added: "osf.b150.v1.0"
